File: wacca_ws2813_rev20240415/wacca_ws2813.kicad_pcb (KiCad board)
At the start: 2 copper layers, 219 x 18 mm, 16 parts, among them CN1 JST XA 3p, CN2 JST XA 3p, CN3 JST XA 4p, U1 1503a, U2 1503a

Commit message: Update revision date
Other:
- board text added: "Rev:20240415"
- board text removed: "Rev:20240408"
Changed lines of the file:
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@@
 		)
 	)
-	(gr_text "Rev:20240408"
+	(gr_text "Rev:20240415"
 		(at 41.935714 106.5 0)
 		(layer "B.SilkS")
